File: Kyosha.kicad_pcb (KiCad board)
At the start: 2 copper layers, 220.3 x 58.3 mm, 64 parts, among them SW1 SW_PUSH, SW10 SW_PUSH, SW11 SW_PUSH, SW12 SW_PUSH, SW13 SW_PUSH, SW14 SW_PUSH, SW15 SW_PUSH, SW16 SW_PUSH, SW17 SW_PUSH, SW18 SW_PUSH, SW19 SW_PUSH, SW2 SW_PUSH, SW20 SW_PUSH, SW21 SW_PUSH, SW22 SW_PUSH, SW23 SW_PUSH, SW24 SW_PUSH, SW25 SW_PUSH, SW26 SW_PUSH, SW27 SW_PUSH, SW28 SW_PUSH, SW29 SW_PUSH, SW3 SW_PUSH, SW30 SW_PUSH, SW31 SW_PUSH, SW32 SW_PUSH, SW4 SW_PUSH, SW5 SW_PUSH, SW6 SW_PUSH, SW7 SW_PUSH, SW8 SW_PUSH, SW9 SW_PUSH, U1 ProMicro

Commit message: pcb first pass
Connections:
- U1 pad 1: Net-(U1-Pad1) -> col0
- U1 pad 10: col5 -> Net-(U1-Pad10)
- U1 pad 11: col6 -> col7
- U1 pad 12: col7 -> col6
- U1 pad 17: col4 -> Net-(U1-Pad17)
- U1 pad 18: col3 -> col1
- U1 pad 19: col2 -> row1
- U1 pad 2: Net-(U1-Pad2) -> row2
- U1 pad 20: Net-(U1-Pad20) -> row0
- U1 pad 5: col0 -> col2
- U1 pad 6: col1 -> col3
- U1 pad 7: row0 -> col4
- U1 pad 8: row1 -> col5
- U1 pad 9: row2 -> Net-(U1-Pad9)
Routing:
- net col10: track 0.00 -> 224.9 mm
- net col9: track 0.00 -> 196.9 mm
- net row0: track 0.00 -> 196.0 mm, vias 0 -> 10
- net row1: track 0.00 -> 194.7 mm, vias 0 -> 11
- net row2: track 0.00 -> 187.7 mm, vias 0 -> 9
- net col8: track 0.00 -> 173.4 mm
- net col7: track 0.00 -> 159.5 mm, vias 0 -> 1
- net col6: track 0.00 -> 137.6 mm, vias 0 -> 1
- net col5: track 0.00 -> 128.4 mm, vias 0 -> 1
- net col4: track 0.00 -> 112.4 mm, vias 0 -> 1
- net col3: track 0.00 -> 96.5 mm, vias 0 -> 1
- net col2: track 0.00 -> 80.5 mm, vias 0 -> 1
- net col0: track 0.00 -> 56.7 mm
- net col1: track 0.00 -> 54.7 mm, vias 0 -> 1
- net GND: track 0.00 -> 32.1 mm
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- added copper zone on B.Cu, net GND
- added copper zone on F.Cu, net GND
